Commit message: Added some basic Gazebo material color implementation and adjusted servo rotation axis values

File: description/materials.xacro (robot description, xacro)
@@ -18,4 +18,7 @@
         <!-- 18 18 36 inches for the max size hull box-->
         <!-- keep in mind ROS uses metric -->
+    <xacro:property name="nasa_hull_length" value="0.4572" />
+    <xacro:property name="nasa_hull_width" value="0.4572" />
+    <xacro:property name="nasa_hull_height" value="0.9144" />
     <xacro:property name="hull_length" value="0.4572" />
     <xacro:property name="hull_width" value="0.4572" />

File: description/robot_core.xacro (robot description, xacro)
@@ -7,5 +7,5 @@
     <<link name="base_link">
     </link>
-    <!-- HULL LINK -->
+    <!-- HULL LINK ===========================================-->
     <<joint name="hull_joint" type="fixed">
         <parent link="base_link"/>
@@ -23,4 +23,5 @@
         </visual>
         <<collision>
+            <!-- for now, make the colission geomentry the same as the basic box shape -->
             <<origin xyz="0.1 0.0 0.5" rpy = "0.0 0.0 0.0"/>
             <<geometry>
@@ -32,5 +33,8 @@
         </xacro:inertial_box>
     <link/>
-    <!-- MOTOR LINK -->>
+    <gazebo reference="hull">
+    <material>Gazebo/orange</material> <!--Do we need to add a materuak section to the launch file now?-->
+    </gazebo>
+    <!-- MOTOR LINK ===========================================-->>
         <!--the motor and servo link will probably need the joint state publisher gui to be seen-->
     <joint name="motor_joint" type="continuous">
@@ -49,11 +53,14 @@
         </visual>
     </link>
-    <!-- SERVO LINK -->>
+    <gazebo reference="motor">
+    <material>Gazebo/blue</material>
+    </gazebo>
+    <!-- SERVO LINK ===========================================-->>
     <joint name="servo_joint" type="continuous">
         <parent link="base_link"/>
         <child link="servo"/>
         <<origin xyz="0.2 0.0 0.0" rpy="0.0 0.0 0.0"/>
-        <!-- "CW forward CCW backward" -Eric -->
-        <<axis xyz="0.0 0.0 1.0"/>
+        <!-- "Right is clockwise" -->
+        <<axis xyz="0.0 1.0 0.0"/>
     <joint/>
     <<link name="servo">
@@ -65,5 +72,8 @@
         </visual>
     </link>
-    <!-- TRNSMISSION --> <!--fix, may not be needed...-->>
+    <gazebo reference="servo">
+    <material>Gazebo/green</material>
+    </gazebo>
+    <!-- TRNSMISSION ===========================================--> <!--fix, may not be needed...-->>
     <transmission name="rudder_trans">
         <type>transmission_interface/SimpleTransmission</type>

Commit message: fixed XML errors

File: description/materials.xacro (robot description, xacro)
@@ -1,17 +1,17 @@
 <?xml version="1.0"?>
-<robot xmls:xacro="http://ww.ros.org/wiki/xacro" >
+<robot xmlns:xacro="http://ww.ros.org/wiki/xacro" >
     <!-- Color Material Section -->>
-    <<material name="white">
-        <<color rgba="1 1 1 1"/>
-    </material>>
-    <<material name="orange">
-        <<color rgba="1 0.5 0 1"/>
-    </material>>
-    <<material name="blue">
-        <<color rgba="0 0 1 1"/>
-    </material>>
-    <<material name="green">
-        <<color rgba="0 1 .1 1"/>
-    </material>>
+    <material name="white">
+        <color rgba="1 1 1 1"/>
+    </material>
+    <material name="orange">
+        <color rgba="1 0.5 0 1"/>
+    </material>
+    <material name="blue">
+        <color rgba="0 0 1 1"/>
+    </material>
+    <material name="green">
+        <color rgba="0 1 .1 1"/>
+    </material>
     <!-- PROPERTIE VARIABLES -->
     <!--Hull Size-->>

Commit message: Added Simple Antenna Variables and an implementation of their shape and links in the robot core file

File: description/materials.xacro (robot description, xacro)
@@ -2,14 +2,14 @@
 <robot xmlns:xacro="http://ww.ros.org/wiki/xacro" >
     <!-- Color Material Section -->>
-    <material name="white">
+    <material name="white">             <!--hull color-->
         <color rgba="1 1 1 1"/>
     </material>
-    <material name="orange">
+    <material name="orange">            <!--servo color-->
         <color rgba="1 0.5 0 1"/>
     </material>
-    <material name="blue">
+    <material name="blue">              <!--antenna color-->
         <color rgba="0 0 1 1"/>
     </material>
-    <material name="green">
+    <material name="green">             <!--motor color-->
         <color rgba="0 1 .1 1"/>
     </material>
@@ -25,3 +25,10 @@
     <xacro:property name="hull_height" value="0.9144" />
     <xacro:property name="CRAFT_mass" value="2.5" />
+    <!-- ANTENNA VARIABLES -->
+        <!-- Not Final Values, need to calculate these with Tyler -->
+    <xacro:property name="lamda" value="0.125" />
+    <xacro:property name="antenna_height" value="0.225" />
+    <xacro:property name="antenna_spacing" value="0.250" /> <!--use for both x and z((?), is it y? its the flat coordinates, not the height)-->
+    <xacro:property name="antenna_center_offset" value="0.110" /> <!--offset for antenna center joint to be in correct destination-->
+    <xacro:property name="antenna_radius" value="0.075" />
 </robot>

File: description/robot_core.xacro (robot description, xacro)
@@ -86,3 +86,73 @@
         </actuator>
     </transmission>
+    <!-- ANTENNA SECTION ============================================================================-->
+    <!-- the antennas are position as following:
+                    Front
+                      ^
+            Left |  4   1  |  Right
+                 |  3   2  |
+                    _____
+                     Back
+            Y
+            |_X
+          Z/
+    -->
+    <joint name="antenna_center_joint" type="fixed">
+        <parent link="base_link"/>
+        <child link="antenna_center"/>
+        <origin xyz="${hull_length/2 - antenna_center_offset} ${hull_length} 0.0"/> <!--I think base_link is centered on the otooom, so the nase antenna center should be UP and more forward-->
+    </joint>
+    <joint name="antenna_1_joint" type="fixed">
+        <parent link="antenna_center"/>
+        <child link="antenna_1"/>
+        <origin xyz="${antenna_spacing} 0.0 ${antenna_spacing}"/> <!--I think base_link is centered on the otooom, so the nase antenna center should be UP and more forward-->
+    </joint>
+    <joint name="antenna_2_joint" type="fixed">
+        <parent link="antenna_center"/>
+        <child link="antenna_2"/>
+        <origin xyz="${antenna_spacing} 0.0 -${antenna_spacing}"/> <!--I think base_link is centered on the otooom, so the nase antenna center should be UP and more forward-->
+    </joint>
+    <joint name="antenna_3_joint" type="fixed">
+        <parent link="antenna_center"/>
+        <child link="antenna_3"/>
+        <origin xyz="-${antenna_spacing} 0.0 -${antenna_spacing}"/> <!--I think base_link is centered on the otooom, so the nase antenna center should be UP and more forward-->
+    </joint>
+    <joint name="antenna_4_joint" type="fixed">
+        <parent link="antenna_center"/>
+        <child link="antenna_4"/>
+        <origin xyz="-${antenna_spacing} 0.0 ${antenna_spacing}"/> <!--I think base_link is centered on the otooom, so the nase antenna center should be UP and more forward-->
+    </joint>
+    <!--Antenna Antenna Extrusions-->
+    <link name="antenna_1">
+        <visual>
+            <geometry>
+                <cylinder radius="${antenna_radius}" length="${antenna_height}"/>
+            </geometry>
+            <material name="blue"/>
+        </visual>
+    </link>
+    <link name="antenna_2">
+        <visual>
+            <geometry>
+                <cylinder radius="${antenna_radius}" length="${antenna_height}"/>
+            </geometry>
+            <material name="blue"/>
+        </visual>
+    </link>
+    <link name="antenna_3">
+        <visual>
+            <geometry>
+                <cylinder radius="${antenna_radius}" length="${antenna_height}"/>
+            </geometry>
+            <material name="blue"/>
+        </visual>
+    </link>
+    <link name="antenna_4">
+        <visual>
+            <geometry>
+                <cylinder radius="${antenna_radius}" length="${antenna_height}"/>
+            </geometry>
+            <material name="blue"/>
+        </visual>
+    </link>
 </robot>

Commit message: Added Gazebo Part coloring and fixed some comments relating to it

File: description/materials.xacro (robot description, xacro)
@@ -2,8 +2,8 @@
 <robot xmlns:xacro="http://ww.ros.org/wiki/xacro" >
     <!-- Color Material Section -->>
-    <material name="white">             <!--hull color-->
+    <material name="white">             <!--servo color-->
         <color rgba="1 1 1 1"/>
     </material>
-    <material name="orange">            <!--servo color-->
+    <material name="orange">            <!--hull color-->
         <color rgba="1 0.5 0 1"/>
     </material>

File: description/robot_core.xacro (robot description, xacro)
@@ -20,5 +20,5 @@
                 <box size="${hull_length} ${hull_width} ${hull_height}"/>
             </geometry>
-            <material name="white"/>
+            <material name="orange"/>
         </visual>
         <collision>
@@ -35,5 +35,5 @@
 	</link>
     <gazebo reference="hull">
-    	<material>Gazebo/orange</material> <!--Do we need to add a materuak section to the launch file now?-->
+    	<material>Gazebo/Orange</material> <!--Do we need to add a material section to the launch file now?-->
     </gazebo>
     <!-- MOTOR LINK ===========================================-->>
@@ -55,5 +55,5 @@
     </link>
     <gazebo reference="motor">
-    	<material>Gazebo/blue</material>
+    	<material>Gazebo/green</material>
     </gazebo>
     <!-- SERVO LINK ===========================================-->>
@@ -70,9 +70,9 @@
                 <cylinder radius="0.2" length="0.1"/>
             </geometry>
-            <material name="orange"/>
+            <material name="white"/>
         </visual>
     </link>
     <gazebo reference="servo">
-    	<material>Gazebo/green</material>
+    	<material>Gazebo/White</material>
     </gazebo>
     <!-- TRNSMISSION ===========================================--> <!--fix, may not be needed...-->>
@@ -123,5 +123,5 @@
         <origin xyz="-${antenna_spacing} 0.0 ${antenna_spacing}"/> <!--I think base_link is centered on the otooom, so the nase antenna center should be UP and more forward-->
     </joint>
-    <!--Antenna Antenna Extrusions-->
+        <!--Antenna Antennai Extrusions-->
     <link name="antenna_1">
         <visual>
@@ -156,3 +156,16 @@
         </visual>
     </link>
+        <!--Gazebo Colors-->
+    <gazebo reference="antenna_1">
+    	<material>Gazebo/Blue</material>
+    </gazebo>
+    <gazebo reference="antenna_2">
+    	<material>Gazebo/Blue</material>
+    </gazebo>
+    <gazebo reference="antenna_3">
+    	<material>Gazebo/Blue</material>
+    </gazebo>
+    <gazebo reference="antenna_4">
+    	<material>Gazebo/Blue</material>
+    </gazebo>
 </robot>

Commit message: Added a basic control xacro file from the articulated robotics blog, This mauy cause launch errors, and more parameters were added

File: description/materials.xacro (robot description, xacro)
@@ -25,4 +25,8 @@
     <xacro:property name="hull_height" value="0.9144" />
     <xacro:property name="CRAFT_mass" value="2.5" />
+    <xacro:property name="motor_radius" value="0.15" />
+    <xacro:property name="servo_radius" value="0.24" />
+    <xacro:property name="motor_length" value="0.65" />
+    <xacro:property name="servo_length" value="0.20" />
     <!-- ANTENNA VARIABLES -->
         <!-- Not Final Values, need to calculate these with Tyler -->

File: description/robot_core.xacro (robot description, xacro)
@@ -49,5 +49,5 @@
         <visual>
             <geometry>
-                <cylinder radius="0.15" length="0.3"/>
+                <cylinder radius="${motor_radius}" length="${motor_length}"/>
             </geometry>
             <material name="green"/>
@@ -62,5 +62,5 @@
         <child link="servo"/>
         <origin xyz="0.2 0.0 0.0" rpy="0.0 0.0 0.0"/>
-        <!-- "Right is clockwise" -->
+        <!-- "Turning right is clockwise" -->
         <axis xyz="0.0 1.0 0.0"/>
     </joint>
@@ -68,5 +68,5 @@
         <visual>
             <geometry>
-                <cylinder radius="0.2" length="0.1"/>
+                <cylinder radius="${servo_radius}" length="${servo_length}"/>
             </geometry>
             <material name="white"/>

Commit message: reverted 6 commits effecting XML that should be in a branch

File: description/materials.xacro (robot description, xacro)
@@ -2,8 +2,8 @@
 <robot xmlns:xacro="http://ww.ros.org/wiki/xacro" >
     <!-- Color Material Section -->>
-    <material name="white">             <!--servo color-->
+    <material name="white">             <!--hull color-->
         <color rgba="1 1 1 1"/>
     </material>
-    <material name="orange">            <!--hull color-->
+    <material name="orange">            <!--servo color-->
         <color rgba="1 0.5 0 1"/>
     </material>
@@ -25,8 +25,4 @@
     <xacro:property name="hull_height" value="0.9144" />
     <xacro:property name="CRAFT_mass" value="2.5" />
-    <xacro:property name="motor_radius" value="0.15" />
-    <xacro:property name="servo_radius" value="0.24" />
-    <xacro:property name="motor_length" value="0.65" />
-    <xacro:property name="servo_length" value="0.20" />
     <!-- ANTENNA VARIABLES -->
         <!-- Not Final Values, need to calculate these with Tyler -->

File: description/robot.urdf.xacro (robot description, xacro)
@@ -2,4 +2,3 @@
 <robot xmlns:xacro="http://www.ros.org/wiki/xacro"  name="robot">
     <xacro:include filename="robot_core.xacro" />
-    <xacro:include filename="gazebo_control.xacro" />
 </robot>

File: description/robot_core.xacro (robot description, xacro)
@@ -20,5 +20,5 @@
                 <box size="${hull_length} ${hull_width} ${hull_height}"/>
             </geometry>
-            <material name="orange"/>
+            <material name="white"/>
         </visual>
         <collision>
@@ -29,13 +29,11 @@
             </geometry>
         </collision>
-		<!-- TODO define the mass here - using placeholder 1.5 kg, add CRAFT_mass to mass when not chencking -->
-        <xacro:inertial_box mass="1.5" x="${hull_length}" y="${hull_width}" z="${hull_height}">
-            <origin xyz="0.1 0.0 0.0" rpy = "0.0 0.0 0.0"/>
+		<!-- TODO define the mass here - using placeholder 1.5 kg -->
+        <xacro:inertial_box mass="1.5" x="0.1" y="0.0" z="0.5">
+            <origin xyz="0.0 0.0 0.0" />
         </xacro:inertial_box>
 	</link>
     <gazebo reference="hull">
-    	<material>Gazebo/Orange</material> <!--Do we need to add a material section to the launch file now?-->
-        <mu1 = "0.0001"/>
-        <mu2 = "0.0001"/> <!--these are both needed for the lack of friction-->
+    	<material>Gazebo/orange</material> <!--Do we need to add a materuak section to the launch file now?-->
     </gazebo>
     <!-- MOTOR LINK ===========================================-->>
@@ -51,5 +49,5 @@
         <visual>
             <geometry>
-                <cylinder radius="${motor_radius}" length="${motor_length}"/>
+                <cylinder radius="0.15" length="0.3"/>
             </geometry>
             <material name="green"/>
@@ -57,5 +55,5 @@
     </link>
     <gazebo reference="motor">
-    	<material>Gazebo/green</material>
+    	<material>Gazebo/blue</material>
     </gazebo>
     <!-- SERVO LINK ===========================================-->>
@@ -64,5 +62,5 @@
         <child link="servo"/>
         <origin xyz="0.2 0.0 0.0" rpy="0.0 0.0 0.0"/>
-        <!-- "Turning right is clockwise" -->
+        <!-- "Right is clockwise" -->
         <axis xyz="0.0 1.0 0.0"/>
     </joint>
@@ -70,11 +68,11 @@
         <visual>
             <geometry>
-                <cylinder radius="${servo_radius}" length="${servo_length}"/>
+                <cylinder radius="0.2" length="0.1"/>
             </geometry>
-            <material name="white"/>
+            <material name="orange"/>
         </visual>
     </link>
     <gazebo reference="servo">
-    	<material>Gazebo/White</material>
+    	<material>Gazebo/green</material>
     </gazebo>
     <!-- TRNSMISSION ===========================================--> <!--fix, may not be needed...-->>
@@ -125,5 +123,5 @@
         <origin xyz="-${antenna_spacing} 0.0 ${antenna_spacing}"/> <!--I think base_link is centered on the otooom, so the nase antenna center should be UP and more forward-->
     </joint>
-        <!--Antenna Antennai Extrusions-->
+    <!--Antenna Antenna Extrusions-->
     <link name="antenna_1">
         <visual>
@@ -158,16 +156,3 @@
         </visual>
     </link>
-        <!--Gazebo Colors-->
-    <gazebo reference="antenna_1">
-    	<material>Gazebo/Blue</material>
-    </gazebo>
-    <gazebo reference="antenna_2">
-    	<material>Gazebo/Blue</material>
-    </gazebo>
-    <gazebo reference="antenna_3">
-    	<material>Gazebo/Blue</material>
-    </gazebo>
-    <gazebo reference="antenna_4">
-    	<material>Gazebo/Blue</material>
-    </gazebo>
 </robot>

Commit message: Revert "Added Simple Antenna Variables and an implementation of their shape and links in the robot core file"
This reverts commit fdb7cfdd86ffccc35b2f982bfae54a92e49d4833.

File: description/materials.xacro (robot description, xacro)
@@ -2,14 +2,14 @@
 <robot xmlns:xacro="http://ww.ros.org/wiki/xacro" >
     <!-- Color Material Section -->>
-    <material name="white">             <!--hull color-->
+    <material name="white">
         <color rgba="1 1 1 1"/>
     </material>
-    <material name="orange">            <!--servo color-->
+    <material name="orange">
         <color rgba="1 0.5 0 1"/>
     </material>
-    <material name="blue">              <!--antenna color-->
+    <material name="blue">
         <color rgba="0 0 1 1"/>
     </material>
-    <material name="green">             <!--motor color-->
+    <material name="green">
         <color rgba="0 1 .1 1"/>
     </material>
@@ -25,10 +25,3 @@
     <xacro:property name="hull_height" value="0.9144" />
     <xacro:property name="CRAFT_mass" value="2.5" />
-    <!-- ANTENNA VARIABLES -->
-        <!-- Not Final Values, need to calculate these with Tyler -->
-    <xacro:property name="lamda" value="0.125" />
-    <xacro:property name="antenna_height" value="0.225" />
-    <xacro:property name="antenna_spacing" value="0.250" /> <!--use for both x and z((?), is it y? its the flat coordinates, not the height)-->
-    <xacro:property name="antenna_center_offset" value="0.110" /> <!--offset for antenna center joint to be in correct destination-->
-    <xacro:property name="antenna_radius" value="0.075" />
 </robot>

File: description/robot_core.xacro (robot description, xacro)
@@ -86,73 +86,3 @@
         </actuator>
     </transmission>
-    <!-- ANTENNA SECTION ============================================================================-->
-    <!-- the antennas are position as following:
-                    Front
-                      ^
-            Left |  4   1  |  Right
-                 |  3   2  |
-                    _____
-                     Back
-            Y
-            |_X
-          Z/
-    -->
-    <joint name="antenna_center_joint" type="fixed">
-        <parent link="base_link"/>
-        <child link="antenna_center"/>
-        <origin xyz="${hull_length/2 - antenna_center_offset} ${hull_length} 0.0"/> <!--I think base_link is centered on the otooom, so the nase antenna center should be UP and more forward-->
-    </joint>
-    <joint name="antenna_1_joint" type="fixed">
-        <parent link="antenna_center"/>
-        <child link="antenna_1"/>
-        <origin xyz="${antenna_spacing} 0.0 ${antenna_spacing}"/> <!--I think base_link is centered on the otooom, so the nase antenna center should be UP and more forward-->
-    </joint>
-    <joint name="antenna_2_joint" type="fixed">
-        <parent link="antenna_center"/>
-        <child link="antenna_2"/>
-        <origin xyz="${antenna_spacing} 0.0 -${antenna_spacing}"/> <!--I think base_link is centered on the otooom, so the nase antenna center should be UP and more forward-->
-    </joint>
-    <joint name="antenna_3_joint" type="fixed">
-        <parent link="antenna_center"/>
-        <child link="antenna_3"/>
-        <origin xyz="-${antenna_spacing} 0.0 -${antenna_spacing}"/> <!--I think base_link is centered on the otooom, so the nase antenna center should be UP and more forward-->
-    </joint>
-    <joint name="antenna_4_joint" type="fixed">
-        <parent link="antenna_center"/>
-        <child link="antenna_4"/>
-        <origin xyz="-${antenna_spacing} 0.0 ${antenna_spacing}"/> <!--I think base_link is centered on the otooom, so the nase antenna center should be UP and more forward-->
-    </joint>
-    <!--Antenna Antenna Extrusions-->
-    <link name="antenna_1">
-        <visual>
-            <geometry>
-                <cylinder radius="${antenna_radius}" length="${antenna_height}"/>
-            </geometry>
-            <material name="blue"/>
-        </visual>
-    </link>
-    <link name="antenna_2">
-        <visual>
-            <geometry>
-                <cylinder radius="${antenna_radius}" length="${antenna_height}"/>
-            </geometry>
-            <material name="blue"/>
-        </visual>
-    </link>
-    <link name="antenna_3">
-        <visual>
-            <geometry>
-                <cylinder radius="${antenna_radius}" length="${antenna_height}"/>
-            </geometry>
-            <material name="blue"/>
-        </visual>
-    </link>
-    <link name="antenna_4">
-        <visual>
-            <geometry>
-                <cylinder radius="${antenna_radius}" length="${antenna_height}"/>
-            </geometry>
-            <material name="blue"/>
-        </visual>
-    </link>
 </robot>
