Commit message: attempted fixE ISSue with minimal example

File: description/robot_urdf_joints.xacro (robot description, xacro)
@@ -9,5 +9,5 @@
 	<joint name="base_link_to_base" type="fixed">
 		<parent link="base_link" />
-		<child link="staticrobot" />
+		<child link="hull" />
 		<origin rpy="0.0 0 0" xyz="0 0 0" />
 	</joint>
