Commit message: added xacro macros of stl files

File: description/physics_include.xacro (robot description, xacro)
@@ -1,7 +1,52 @@
 <?xml version="1.0"?>
 <robot xmlns:xacro="http://www.ros.org/wiki/xacro" >
+	<!-- Include meshes -->
+	<xacro:macro name="30degsplit_mesh">
+        <mesh filename="file://$(find msd_bot)/meshes/30degsplitter.stl" scale="0.001 0.001 0.001"/>
+    </xacro:macro>
+	<xacro:macro name="antenna_mesh">
+        <mesh filename="file://$(find msd_bot)/meshes/antenna.stl" scale="0.001 0.001 0.001"/>
+    </xacro:macro>
+	<xacro:macro name="basedowel_mesh">
+        <mesh filename="file://$(find msd_bot)/meshes/basedowel.stl" scale="0.001 0.001 0.001"/>
+    </xacro:macro>
+	<xacro:macro name="brushlessmotor_mesh">
+		<mesh filename="file://$(find msd_bot)/meshes/brushlessmotor.stl" scale="0.001 0.001 0.001"/>
+	</xacro:macro>
+    <xacro:macro name="cargohold_mesh">
+        <mesh filename="file://$(find msd_bot)/meshes/cargohold.stl" scale="0.001 0.001 0.001"/>
+    </xacro:macro>
+    <xacro:macro name="hull_mesh">
+        <mesh filename="file://$(find msd_bot)/meshes/hull.stl" scale="0.001 0.001 0.001"/>
+    </xacro:macro>
+	<xacro:macro name="hullcover_mesh">
+		<mesh filename="file://$(find msd_bot)/meshes/hullcover.stl" scale="0.001 0.001 0.001"/>
+	</xacro:macro>
+	<xacro:macro name="propeller_mesh">
+		<mesh filename="file://$(find msd_bot)/meshes/propeller.stl" scale="0.001 0.001 0.001"/>
+	</xacro:macro>
+	<xacro:macro name="rudder_mesh">
+		<mesh filename="file://$(find msd_bot)/meshes/rudder.stl" scale="0.001 0.001 0.001"/>
+	</xacro:macro>
+	<xacro:macro name="rudderbottommount_mesh">
+		<mesh filename="file://$(find msd_bot)/meshes/rudderbottommount.stl" scale="0.001 0.001 0.001"/>
+	</xacro:macro>
+	<xacro:macro name="servo_mesh">
+		<mesh filename="file://$(find msd_bot)/meshes/servo.stl" scale="0.001 0.001 0.001"/>
+	</xacro:macro>
+	<xacro:macro name="servomount_mesh">
+		<mesh filename="file://$(find msd_bot)/meshes/servomount.stl" scale="0.001 0.001 0.001"/>
+	</xacro:macro>
+	<xacro:macro name="sidedowel_mesh">
+		<mesh filename="file://$(find msd_bot)/meshes/sidedowel.stl" scale="0.001 0.001 0.001"/>
+	</xacro:macro>
+	<xacro:macro name="sidedowel2_mesh">
+		<mesh filename="file://$(find msd_bot)/meshes/sidedowel2.stl" scale="0.001 0.001 0.001"/>
+	</xacro:macro>
+	<xacro:macro name="vdowelconnector_mesh">
+		<mesh filename="file://$(find msd_bot)/meshes/vdowelconnector.stl" scale="0.001 0.001 0.001"/>
+	</xacro:macro>
     <!-- Specify some standard inertial calculations https://en.wikipedia.org/wiki/List_of_moments_of_inertia -->
     <!-- These make use of xacro's mathematical functionality -->
-    <!-- taken from articuilated robotics -->
     <xacro:macro name="inertial_sphere" params="mass radius *origin">
         <inertial>

Commit message: partially complete better xacro

File: description/physics_include.xacro (robot description, xacro)
@@ -2,5 +2,5 @@
 <robot xmlns:xacro="http://www.ros.org/wiki/xacro" >
 	<!-- Include meshes -->
-	<xacro:macro name="30degsplit_mesh">
+	<xacro:macro name="thirtydegsplitter_mesh">
         <mesh filename="file://$(find msd_bot)/meshes/30degsplitter.stl" scale="0.001 0.001 0.001"/>
     </xacro:macro>
@@ -44,5 +44,5 @@
 		<mesh filename="file://$(find msd_bot)/meshes/sidedowel2.stl" scale="0.001 0.001 0.001"/>
 	</xacro:macro>
-	<xacro:macro name="vdowelconnector_mesh">
+	<xacro:macro name="vdowel_mesh">
 		<mesh filename="file://$(find msd_bot)/meshes/vdowelconnector.stl" scale="0.001 0.001 0.001"/>
 	</xacro:macro>

File: description/robot.urdf.xacro (robot description, xacro)
@@ -1,4 +1,7 @@
 <?xml version="1.0"?>
-<robot xmlns:xacro="http://www.ros.org/wiki/xacro"  name="robot">
-    <xacro:include filename="robot_core.xacro" />
+<robot xmlns:xacro="http://www.ros.org/wiki/xacro"  name="msd_bot">
+    <!-- ***************  CONFIGURE ROBOT'S LINKS  *******************-->
+    <xacro:include filename="robot_urdf_links.xacro" />
+    <!-- ***************  CONFIGURE ROBOT'S JOINTS  *******************-->
+    <xacro:include filename="hyperdog_urdf_joints.xacro" />
 </robot>

Commit message: additional incremental test fixes

File: description/physics_include.xacro (robot description, xacro)
@@ -3,47 +3,47 @@
 	<!-- Include meshes -->
 	<xacro:macro name="thirtydegsplitter_mesh">
-        <mesh filename="file://$(find msd_bot)/meshes/30degsplitter.stl" scale="0.001 0.001 0.001"/>
+        <mesh filename="file://$(find msd_bot)/meshes/30degsplitter.stl"  />
     </xacro:macro>
 	<xacro:macro name="antenna_mesh">
-        <mesh filename="file://$(find msd_bot)/meshes/antenna.stl" scale="0.001 0.001 0.001"/>
+        <mesh filename="file://$(find msd_bot)/meshes/antenna.stl"  />
     </xacro:macro>
 	<xacro:macro name="basedowel_mesh">
-        <mesh filename="file://$(find msd_bot)/meshes/basedowel.stl" scale="0.001 0.001 0.001"/>
+        <mesh filename="file://$(find msd_bot)/meshes/basedowel.stl"  />
     </xacro:macro>
 	<xacro:macro name="brushlessmotor_mesh">
-		<mesh filename="file://$(find msd_bot)/meshes/brushlessmotor.stl" scale="0.001 0.001 0.001"/>
+		<mesh filename="file://$(find msd_bot)/meshes/brushlessmotor.stl"  />
 	</xacro:macro>
     <xacro:macro name="cargohold_mesh">
-        <mesh filename="file://$(find msd_bot)/meshes/cargohold.stl" scale="0.001 0.001 0.001"/>
+        <mesh filename="file://$(find msd_bot)/meshes/cargohold.stl"  />
     </xacro:macro>
     <xacro:macro name="hull_mesh">
-        <mesh filename="file://$(find msd_bot)/meshes/hull.stl" scale="0.001 0.001 0.001"/>
+        <mesh filename="file://$(find msd_bot)/meshes/hull.stl"  />
     </xacro:macro>
 	<xacro:macro name="hullcover_mesh">
-		<mesh filename="file://$(find msd_bot)/meshes/hullcover.stl" scale="0.001 0.001 0.001"/>
+		<mesh filename="file://$(find msd_bot)/meshes/hullcover.stl"  />
 	</xacro:macro>
 	<xacro:macro name="propeller_mesh">
-		<mesh filename="file://$(find msd_bot)/meshes/propeller.stl" scale="0.001 0.001 0.001"/>
+		<mesh filename="file://$(find msd_bot)/meshes/propeller.stl"  />
 	</xacro:macro>
 	<xacro:macro name="rudder_mesh">
-		<mesh filename="file://$(find msd_bot)/meshes/rudder.stl" scale="0.001 0.001 0.001"/>
+		<mesh filename="file://$(find msd_bot)/meshes/rudder.stl"  />
 	</xacro:macro>
 	<xacro:macro name="rudderbottommount_mesh">
-		<mesh filename="file://$(find msd_bot)/meshes/rudderbottommount.stl" scale="0.001 0.001 0.001"/>
+		<mesh filename="file://$(find msd_bot)/meshes/rudderbottommount.stl"  />
 	</xacro:macro>
 	<xacro:macro name="servo_mesh">
-		<mesh filename="file://$(find msd_bot)/meshes/servo.stl" scale="0.001 0.001 0.001"/>
+		<mesh filename="file://$(find msd_bot)/meshes/servo.stl"  />
 	</xacro:macro>
 	<xacro:macro name="servomount_mesh">
-		<mesh filename="file://$(find msd_bot)/meshes/servomount.stl" scale="0.001 0.001 0.001"/>
+		<mesh filename="file://$(find msd_bot)/meshes/servomount.stl"  />
 	</xacro:macro>
 	<xacro:macro name="sidedowel_mesh">
-		<mesh filename="file://$(find msd_bot)/meshes/sidedowel.stl" scale="0.001 0.001 0.001"/>
+		<mesh filename="file://$(find msd_bot)/meshes/sidedowel.stl"  />
 	</xacro:macro>
 	<xacro:macro name="sidedowel2_mesh">
-		<mesh filename="file://$(find msd_bot)/meshes/sidedowel2.stl" scale="0.001 0.001 0.001"/>
+		<mesh filename="file://$(find msd_bot)/meshes/sidedowel2.stl"  />
 	</xacro:macro>
 	<xacro:macro name="vdowel_mesh">
-		<mesh filename="file://$(find msd_bot)/meshes/vdowelconnector.stl" scale="0.001 0.001 0.001"/>
+		<mesh filename="file://$(find msd_bot)/meshes/vdowelconnector.stl"  />
 	</xacro:macro>
     <!-- Specify some standard inertial calculations https://en.wikipedia.org/wiki/List_of_moments_of_inertia -->

File: description/robot_gazebo.xacro (robot description, xacro)
@@ -14,5 +14,5 @@
         <material>Gazebo/DarkGrey  </material>
     </gazebo>
-    <gazebo reference="staticrobot">
+    <gazebo reference="hull">
         <material>Gazebo/Blue</material>
     </gazebo>

Commit message: made hull appear for vscode ROS

File: description/physics_include.xacro (robot description, xacro)
@@ -3,47 +3,47 @@
 	<!-- Include meshes -->
 	<xacro:macro name="thirtydegsplitter_mesh">
-        <mesh filename="file://$(find msd_bot)/meshes/30degsplitter.stl"  />
+		<mesh filename="package://msd_bot/meshes/30degsplitter.stl"/>
     </xacro:macro>
 	<xacro:macro name="antenna_mesh">
-        <mesh filename="file://$(find msd_bot)/meshes/antenna.stl"  />
+        <mesh filename="package://msd_bot/meshes/antenna.stl"  />
     </xacro:macro>
 	<xacro:macro name="basedowel_mesh">
-        <mesh filename="file://$(find msd_bot)/meshes/basedowel.stl"  />
+        <mesh filename="package://msd_bot/meshes/basedowel.stl"  />
     </xacro:macro>
 	<xacro:macro name="brushlessmotor_mesh">
-		<mesh filename="file://$(find msd_bot)/meshes/brushlessmotor.stl"  />
+		<mesh filename="package://msd_bot/meshes/brushlessmotor.stl"  />
 	</xacro:macro>
     <xacro:macro name="cargohold_mesh">
-        <mesh filename="file://$(find msd_bot)/meshes/cargohold.stl"  />
+        <mesh filename="package://msd_bot/meshes/cargohold.stl"  />
     </xacro:macro>
     <xacro:macro name="hull_mesh">
-        <mesh filename="file://$(find msd_bot)/meshes/hull.stl"  />
+        <mesh filename="package://msd_bot/meshes/hull.stl"  />
     </xacro:macro>
 	<xacro:macro name="hullcover_mesh">
-		<mesh filename="file://$(find msd_bot)/meshes/hullcover.stl"  />
+		<mesh filename="package://msd_bot/meshes/hullcover.stl"  />
 	</xacro:macro>
 	<xacro:macro name="propeller_mesh">
-		<mesh filename="file://$(find msd_bot)/meshes/propeller.stl"  />
+		<mesh filename="package://msd_bot/meshes/propeller.stl"  />
 	</xacro:macro>
 	<xacro:macro name="rudder_mesh">
-		<mesh filename="file://$(find msd_bot)/meshes/rudder.stl"  />
+		<mesh filename="package://msd_bot/meshes/rudder.stl"  />
 	</xacro:macro>
 	<xacro:macro name="rudderbottommount_mesh">
-		<mesh filename="file://$(find msd_bot)/meshes/rudderbottommount.stl"  />
+		<mesh filename="package://msd_bot/meshes/rudderbottommount.stl"  />
 	</xacro:macro>
 	<xacro:macro name="servo_mesh">
-		<mesh filename="file://$(find msd_bot)/meshes/servo.stl"  />
+		<mesh filename="package://msd_bot/meshes/servo.stl"  />
 	</xacro:macro>
 	<xacro:macro name="servomount_mesh">
-		<mesh filename="file://$(find msd_bot)/meshes/servomount.stl"  />
+		<mesh filename="package://msd_bot/meshes/servomount.stl"  />
 	</xacro:macro>
 	<xacro:macro name="sidedowel_mesh">
-		<mesh filename="file://$(find msd_bot)/meshes/sidedowel.stl"  />
+		<mesh filename="package://msd_bot/meshes/sidedowel.stl"  />
 	</xacro:macro>
 	<xacro:macro name="sidedowel2_mesh">
-		<mesh filename="file://$(find msd_bot)/meshes/sidedowel2.stl"  />
+		<mesh filename="package://msd_bot/meshes/sidedowel2.stl"  />
 	</xacro:macro>
 	<xacro:macro name="vdowel_mesh">
-		<mesh filename="file://$(find msd_bot)/meshes/vdowelconnector.stl"  />
+		<mesh filename="package://msd_bot/meshes/vdowelconnector.stl"  />
 	</xacro:macro>
     <!-- Specify some standard inertial calculations https://en.wikipedia.org/wiki/List_of_moments_of_inertia -->
