Commit message: simplified significantly to get minimal simulatable example

File: description/robot.urdf.xacro (robot description, xacro)
@@ -4,4 +4,6 @@
     <xacro:include filename="robot_urdf_links.xacro" />
     <!-- ***************  CONFIGURE ROBOT'S JOINTS  *******************-->
-    <xacro:include filename="hyperdog_urdf_joints.xacro" />
+    <xacro:include filename="robot_urdf_joints.xacro" />
+	<!-- ***************  provide info for Gz  *******************-->
+	<xacro:include filename="robot_gazebo.xacro" />
 </robot>

File: description/robot_urdf_joints.xacro (robot description, xacro)
@@ -12,15 +12,7 @@
 		<origin rpy="0.0 0 0" xyz="0 0 0" />
 	</joint>
-	<!-- *********  propeller  ********* -->
-	<joint name="propeller_shaft" type="revolute">
-		<origin xyz="0.0819412 1.169 0.338466" rpy="1.5708 -1.02461e-33 -3.55271e-15" />
-		<parent link="staticrobot" />
-		<child link="propeller" />
-		<axis xyz="0 0 1" />
-		<limit effort="1" velocity="20" />
-		<joint_properties friction="0.0" />
-	</joint>
+</robot>
     <!-- *********  servo  ********* -->
-	<joint name="servo_rudder" type="revolute">
+	<!-- <joint name="servo_rudder" type="revolute">
 		<origin xyz="0.0819412 1.21345 0.560081" rpy="7.78435e-16 6.85351e-15 0.0697974" />
 		<parent link="staticrobot" />
@@ -30,3 +22,3 @@
 		<joint_properties friction="0.0" />
 	</joint>
-</robot>
+</robot> -->

File: description/robot_urdf_links.xacro (robot description, xacro)
@@ -9,9 +9,30 @@
     <xacro:include filename="physics_include.xacro" />
 	<link name="base_link"></link>
-	<link name="staticrobot">
+	<link name="hull">
+		<visual>
+			<origin xyz="0.0819412 0.783555 0.478166" rpy="0 -0 0" />
+			<geometry>
+				<xacro:hull_mesh></xacro:hull_mesh>
+			</geometry>
+			<material name="hull_material">
+				<color rgba="0.498039 0.498039 0.498039 1.0" />
+			</material>
+		</visual>
+		<collision>
+			<origin xyz="0.0819412 0.783555 0.478166" rpy="0 -0 0" />
+			<geometry>
+				<xacro:hull_mesh></xacro:hull_mesh>
+			</geometry>
+			<material name="hull_material">
+				<color rgba="0.498039 0.498039 0.498039 1.0" />
+			</material>
+		</collision>
+	</link>
+</robot>
+	<!-- <link name="staticrobot">
 		<visual>
 			<origin xyz="-0.0760565 1.12963 0.380489" rpy="0.610865 -1.66533e-16 1.5708" />
 			<geometry>
-				<xacro:vdowelconnector_mesh></xacro:vdowelconnector_mesh>
+				<xacro:vdowel_mesh></xacro:vdowel_mesh>
 			</geometry>
 			<material name="vdowelconnector_material">
@@ -19,10 +40,4 @@
 			</material>
 		</visual>
-		<!-- <collision>
-			<origin xyz="-0.0760565 1.12963 0.380489" rpy="0.610865 -1.66533e-16 1.5708" />
-			<geometry>
-				<xacro:vdowelconnector_mesh></xacro:vdowelconnector_mesh>
-			</geometry>
-		</collision> -->
 		<visual>
 			<origin xyz="0.234341 1.0166 0.558811" rpy="0 -0 0" />
@@ -34,10 +49,4 @@
 			</material>
 		</visual>
-		<!-- <collision>
-			<origin xyz="0.234341 1.0166 0.558811" rpy="0 -0 0" />
-			<geometry>
-				<xacro:antenna_mesh></xacro:antenna_mesh>
-			</geometry>
-		</collision> -->
 		<visual>
 			<origin xyz="0.0819412 1.1436 0.249566" rpy="0 3.15544e-30 -3.14159" />
@@ -49,10 +58,4 @@
 			</material>
 		</visual>
-		<!-- <collision>
-			<origin xyz="0.0819412 1.1436 0.249566" rpy="0 3.15544e-30 -3.14159" />
-			<geometry>
-				<mesh filename="package://msd_bot/rudderbottommount.stl" />
-			</geometry>
-		</collision> -->
 		<visual>
 			<origin xyz="0.0719412 1.22345 0.602081" rpy="-1.5708 6.8762e-15 -1.61338e-29" />
@@ -64,10 +67,4 @@
 			</material>
 		</visual>
-		<!-- <collision>
-			<origin xyz="0.0719412 1.22345 0.602081" rpy="-1.5708 6.8762e-15 -1.61338e-29" />
-			<geometry>
-				<xacro:servo_mesh></xacro:servo_mesh>
-			</geometry>
-		</collision> -->
 		<visual>
 			<origin xyz="0.0819412 0.783555 0.478166" rpy="0 -0 0" />
@@ -97,10 +94,4 @@
 			</material>
 		</visual>
-		<!-- <collision>
-			<origin xyz="0.0819412 1.11217 0.260168" rpy="0 -0 3.14159" />
-			<geometry>
-				<xacro:thirtydegsplitter_mesh></xacro:thirtydegsplitter_mesh>
-			</geometry>
-		</collision> -->
 		<visual>
 			<origin xyz="0.0819412 0.788 0.554366" rpy="0 -0 0" />
@@ -112,10 +103,4 @@
 			</material>
 		</visual>
-		<!-- <collision>
-			<origin xyz="0.0819412 0.788 0.554366" rpy="0 -0 0" />
-			<geometry>
-				<xacro:hullcover_mesh></xacro:hullcover_mesh>
-			</geometry>
-		</collision> -->
 		<visual>
 			<origin xyz="-0.0708549 1.12963 0.376847" rpy="2.53073 -0 -1.5708" />
@@ -127,10 +112,4 @@
 			</material>
 		</visual>
-		<!-- <collision>
-			<origin xyz="-0.0708549 1.12963 0.376847" rpy="2.53073 -0 -1.5708" />
-			<geometry>
-				<xacro:sidedowel_mesh></xacro:sidedowel_mesh>
-			</geometry>
-		</collision> -->
 		<visual>
 			<origin xyz="-0.0704588 1.0166 0.558811" rpy="0 -0 0" />
@@ -142,10 +121,4 @@
 			</material>
 		</visual>
-		<!-- <collision>
-			<origin xyz="-0.0704588 1.0166 0.558811" rpy="0 -0 0" />
-			<geometry>
-				<xacro:antenna_mesh></xacro:antenna_mesh>
-			</geometry>
-		</collision> -->
 		<visual>
 			<origin xyz="0.240157 1.12963 0.380177" rpy="0.610865 5.55112e-17 -1.5708" />
@@ -157,10 +130,4 @@
 			</material>
 		</visual>
-		<!-- <collision>
-			<origin xyz="0.240157 1.12963 0.380177" rpy="0.610865 5.55112e-17 -1.5708" />
-			<geometry>
-				<xacro:vdowel_mesh></xacro:vdowel_mesh>
-			</geometry>
-		</collision> -->
 		<visual>
 			<origin xyz="0.0819412 0.935955 0.401966" rpy="4.36955e-14 2.06286e-14 1.36592e-16" />
@@ -172,10 +139,4 @@
 			</material>
 		</visual>
-		<!-- <collision>
-			<origin xyz="0.0819412 0.935955 0.401966" rpy="4.36955e-14 2.06286e-14 1.36592e-16" />
-			<geometry>
-				<xacro:cargohold_mesh></xacro:cargohold_mesh>
-			</geometry>
-		</collision> -->
 		<visual>
 			<origin xyz="-0.0704588 0.7118 0.558811" rpy="0 -0 0" />
@@ -187,10 +148,4 @@
 			</material>
 		</visual>
-		<!-- <collision>
-			<origin xyz="-0.0704588 0.7118 0.558811" rpy="0 -0 0" />
-			<geometry>
-				<xacro:antenna_mesh></xacro:antenna_mesh>
-			</geometry>
-		</collision> -->
 		<visual>
 			<origin xyz="0.289365 1.12963 0.537786" rpy="1.5708 0.290161 -3.89362e-17" />
@@ -202,10 +157,4 @@
 			</material>
 		</visual>
-		<!-- <collision>
-			<origin xyz="0.289365 1.12963 0.537786" rpy="1.5708 0.290161 -3.89362e-17" />
-			<geometry>
-				<xacro:sidedowel2_mesh></xacro:sidedowel2_mesh>
-			</geometry>
-		</collision> -->
 		<visual>
 			<origin xyz="0.0819412 1.004 0.338466" rpy="3.14159 -0 1.5708" />
@@ -217,10 +166,4 @@
 			</material>
 		</visual>
-		<!-- <collision>
-			<origin xyz="0.0819412 1.004 0.338466" rpy="3.14159 -0 1.5708" />
-			<geometry>
-				<xacro:brushlessmotor_mesh></xacro:brushlessmotor_mesh>
-			</geometry>
-		</collision> -->
 		<visual>
 			<origin xyz="0.234956 1.12963 0.376535" rpy="2.53073 -0 1.5708" />
@@ -232,10 +175,4 @@
 			</material>
 		</visual>
-		<!-- <collision>
-			<origin xyz="0.234956 1.12963 0.376535" rpy="2.53073 -0 1.5708" />
-			<geometry>
-				<xacro:sidedowel_mesh></xacro:sidedowel_mesh>
-			</geometry>
-		</collision> -->
 		<visual>
 			<origin xyz="0.0819412 1.18022 0.574781" rpy="1.45652e-14 6.8762e-15 1.36592e-16" />
@@ -247,10 +184,4 @@
 			</material>
 		</visual>
-		<!-- <collision>
-			<origin xyz="0.0819412 1.18022 0.574781" rpy="1.45652e-14 6.8762e-15 1.36592e-16" />
-			<geometry>
-				<xacro:servomount_mesh></xacro:servomount_mesh>
-			</geometry>
-		</collision> -->
 		<visual>
 			<origin xyz="0.234341 0.7118 0.558811" rpy="0 -0 0" />
@@ -262,10 +193,4 @@
 			</material>
 		</visual>
-		<!-- <collision>
-			<origin xyz="0.234341 0.7118 0.558811" rpy="0 -0 0" />
-			<geometry>
-				<xacro:antenna_mesh></xacro:antenna_mesh>
-			</geometry>
-		</collision> -->
 		<visual>
 			<origin xyz="0.0819412 1.13122 0.260168" rpy="3.14159 -5.55112e-17 3.14159" />
@@ -277,10 +202,4 @@
 			</material>
 		</visual>
-		<!-- <collision>
-			<origin xyz="0.0819412 1.13122 0.260168" rpy="3.14159 -5.55112e-17 3.14159" />
-			<geometry>
-				<xacro:basedowel_mesh></xacro:basedowel_mesh>
-			</geometry>
-		</collision> -->
 		<visual>
 			<origin xyz="-0.125264 1.12963 0.538098" rpy="1.5708 0.290161 3.14159" />
@@ -292,10 +211,4 @@
 			</material>
 		</visual>
-		<!-- <collision>
-			<origin xyz="-0.125264 1.12963 0.538098" rpy="1.5708 0.290161 3.14159" />
-			<geometry>
-				<xacro:sidedowel2_mesh></xacro:sidedowel2_mesh>
-			</geometry>
-		</collision> -->
 		<inertial>
 			<origin xyz="0.0819416 0.933985 0.432327" rpy="0 0 0" />
@@ -351,3 +264,3 @@
 		</inertial>
 	</link>
-</robot>
+</robot> -->

Commit message: consolidated subassems, made working urdf

File: description/robot.urdf.xacro (robot description, xacro)
@@ -1,9 +1,158 @@
 <?xml version="1.0"?>
-<robot xmlns:xacro="http://www.ros.org/wiki/xacro"  name="msd_bot">
-    <!-- ***************  CONFIGURE ROBOT'S LINKS  *******************-->
-    <xacro:include filename="robot_urdf_links.xacro" />
-    <!-- ***************  CONFIGURE ROBOT'S JOINTS  *******************-->
-    <xacro:include filename="robot_urdf_joints.xacro" />
-	<!-- ***************  provide info for Gz  *******************-->
-	<xacro:include filename="robot_gazebo.xacro" />
+<robot xmlns:xacro="http://www.ros.org/wiki/xacro" name="msd_bot">
+<!-- ***************  provide info for Gz  *******************-->
+	<!-- <xacro:include filename="robot_gazebo.xacro" /> -->
+	<link name="base_link"></link>
+	<joint name="base_link_to_base" type="fixed">
+		<parent link="base_link" />
+		<child link="hullassm" />
+		<origin rpy="0.0 0 0" xyz="0 0 0" />
+	</joint>
+	<link name="hullassm">
+		<visual>
+			<origin xyz="0 0 0" rpy="0 -0 0" />
+			<geometry>
+				<mesh filename="package://msd_bot/meshes/hullassm.stl" />
+			</geometry>
+			<material name="hullassm_material">
+				<color rgba="0.24291 0.244006 0.250091 1.0" />
+			</material>
+		</visual>
+		<collision>
+			<origin xyz="0 0 0" rpy="0 -0 0" />
+			<geometry>
+				<mesh filename="package://msd_bot/meshes/hullassm.stl" />
+			</geometry>
+		</collision>
+		<inertial>
+			<origin xyz="1.0307e-06 0.188008 0.124094" rpy="0 0 0" />
+			<mass value="6.29782" />
+			<inertia ixx="0.216502" ixy="-1.02604e-06" ixz="1.28468e-06" iyy="0.0821502"
+				iyz="0.0297739" izz="0.237496" />
+		</inertial>
+	</link>
+	<link name="propeller">
+		<visual>
+			<origin xyz="0 0 0" rpy="0 -0 0" />
+			<geometry>
+				<mesh filename="package://msd_bot/meshes/propeller.stl" />
+			</geometry>
+			<material name="propeller_material">
+				<color rgba="0.682353 0.333333 0.737255 1.0" />
+			</material>
+		</visual>
+		<collision>
+			<origin xyz="0 0 0" rpy="0 -0 0" />
+			<geometry>
+				<mesh filename="package://msd_bot/meshes/propeller.stl" />
+			</geometry>
+		</collision>
+		<inertial>
+			<origin xyz="1.6644e-07 -8.74972e-08 -0.00131544" rpy="0 0 0" />
+			<mass value="0.0252682" />
+			<inertia ixx="1.02998e-05" ixy="4.84789e-11" ixz="7.4214e-11" iyy="1.02998e-05"
+				iyz="5.65357e-11" izz="1.394e-05" />
+		</inertial>
+	</link>
+	<joint name="propeller_shaft" type="continuous">
+		<origin xyz="-2.11292e-18 0.385445 0.0889" rpy="1.5708 -0.187437 -3.49069e-15" />
+		<parent link="hullassm" />
+		<child link="propeller" />
+		<axis xyz="0 0 1" />
+		<limit effort="1" velocity="20" />
+		<joint_properties friction="0.0" />
+	</joint>
+	<link name="topassm">
+		<visual>
+			<origin xyz="0 0 0" rpy="0 -0 0" />
+			<geometry>
+				<mesh filename="package://msd_bot/meshes/topassm.stl" />
+			</geometry>
+			<material name="topassm_material">
+				<color rgba="0.780424 0.75747 0.695877 1.0" />
+			</material>
+		</visual>
+		<collision>
+			<origin xyz="0 0 0" rpy="0 -0 0" />
+			<geometry>
+				<mesh filename="package://msd_bot/meshes/topassm.stl" />
+			</geometry>
+		</collision>
+		<inertial>
+			<origin xyz="0.2286 -0.367849 0.00346183" rpy="0 0 0" />
+			<mass value="0.69925" />
+			<inertia ixx="0.028029" ixy="-2.71051e-19" ixz="-2.03288e-20" iyy="0.0137782"
+				iyz="-7.66504e-05" izz="0.0417123" />
+		</inertial>
+	</link>
+	<joint name="hull_cover" type="fixed">
+		<origin xyz="-0.2286 0.360045 0.3048" rpy="0 3.08149e-32 -4.62274e-32" />
+		<parent link="hullassm" />
+		<child link="topassm" />
+		<axis xyz="0 0 1" />
+		<limit effort="1" velocity="20" />
+		<joint_properties friction="0.0" />
+	</joint>
+	<link name="servocargoassm">
+		<visual>
+			<origin xyz="0 0 0" rpy="0 -0 0" />
+			<geometry>
+				<mesh filename="package://msd_bot/meshes/servocargoassm.stl" />
+			</geometry>
+			<material name="servocargoassm_material">
+				<color rgba="0.621357 0.806496 0.907144 1.0" />
+			</material>
+		</visual>
+		<collision>
+			<origin xyz="0 0 0" rpy="0 -0 0" />
+			<geometry>
+				<mesh filename="package://msd_bot/meshes/servocargoassm.stl" />
+			</geometry>
+		</collision>
+		<inertial>
+			<origin xyz="-2.57314e-10 0.0877782 -0.220495" rpy="0 0 0" />
+			<mass value="8.22292" />
+			<inertia ixx="0.17107" ixy="-2.11808e-10" ixz="6.43831e-10" iyy="0.215272"
+				iyz="0.00150393" izz="0.0855135" />
+		</inertial>
+	</link>
+	<link name="rudder">
+		<visual>
+			<origin xyz="0 0 0" rpy="0 -0 0" />
+			<geometry>
+				<mesh filename="package://msd_bot/meshes/rudder.stl" />
+			</geometry>
+			<material name="rudder_material">
+				<color rgba="0.980392 0.796078 0.262745 1.0" />
+			</material>
+		</visual>
+		<collision>
+			<origin xyz="0 0 0" rpy="0 -0 0" />
+			<geometry>
+				<mesh filename="package://msd_bot/meshes/rudder.stl" />
+			</geometry>
+		</collision>
+		<inertial>
+			<origin xyz="1.73472e-17 0.00323547 -0.179304" rpy="0 0 0" />
+			<mass value="0.0651203" />
+			<inertia ixx="0.000500832" ixy="3.75168e-21" ixz="6.55605e-23" iyy="0.00049688"
+				iyz="1.16286e-05" izz="4.87634e-06" />
+		</inertial>
+	</link>
+	<joint name="servo_rudder" type="continuous">
+		<origin xyz="3.43338e-16 -0.005715 0.074295" rpy="1.5708 1.43827 -1.03735e-13" />
+		<parent link="servocargoassm" />
+		<child link="rudder" />
+		<axis xyz="0 0 1" />
+		<limit effort="1" velocity="20" />
+		<joint_properties friction="0.0" />
+	</joint>
+	<joint name="hull_cargo" type="fixed">
+		<origin xyz="-2.77556e-17 0.3556 0.3048" rpy="-1.5708 -0 -4.62274e-32" />
+		<parent link="hullassm" />
+		<child link="servocargoassm" />
+		<axis xyz="0 0 1" />
+		<limit effort="1" velocity="20" />
+		<joint_properties friction="0.0" />
+	</joint>
 </robot>

Commit message: updated gazebo color tags

File: description/robot.urdf.xacro (robot description, xacro)
@@ -1,6 +1,4 @@
 <?xml version="1.0"?>
 <robot xmlns:xacro="http://www.ros.org/wiki/xacro" name="msd_bot">
-<!-- ***************  provide info for Gz  *******************-->
-	<!-- <xacro:include filename="robot_gazebo.xacro" /> -->
 	<link name="base_link"></link>
 	<joint name="base_link_to_base" type="fixed">
@@ -32,4 +30,7 @@
 		</inertial>
 	</link>
+	<gazebo reference="hullassm">
+        <material>Gazebo/DarkGrey  </material>
+    </gazebo>
 	<link name="propeller">
 		<visual>
@@ -55,4 +56,7 @@
 		</inertial>
 	</link>
+	<gazebo reference="propeller">
+        <material>Gazebo/Purple  </material>
+    </gazebo>
 	<joint name="propeller_shaft" type="continuous">
 		<origin xyz="-2.11292e-18 0.385445 0.0889" rpy="1.5708 -0.187437 -3.49069e-15" />
@@ -86,4 +90,7 @@
 		</inertial>
 	</link>
+	<gazebo reference="topassm">
+        <material>Gazebo/White </material>
+    </gazebo>
 	<joint name="hull_cover" type="fixed">
 		<origin xyz="-0.2286 0.360045 0.3048" rpy="0 3.08149e-32 -4.62274e-32" />
@@ -117,4 +124,7 @@
 		</inertial>
 	</link>
+	<gazebo reference="servocargoassm">
+        <material>Gazebo/LightBlue  </material>
+    </gazebo>
 	<link name="rudder">
 		<visual>
@@ -140,4 +150,7 @@
 		</inertial>
 	</link>
+	<gazebo reference="rudder">
+        <material>Gazebo/Yellow  </material>
+    </gazebo>
 	<joint name="servo_rudder" type="continuous">
 		<origin xyz="3.43338e-16 -0.005715 0.074295" rpy="1.5708 1.43827 -1.03735e-13" />

Commit message: changed links to meshes for Gazebo to work

File: description/robot.urdf.xacro (robot description, xacro)
@@ -11,5 +11,5 @@
 			<origin xyz="0 0 0" rpy="0 -0 0" />
 			<geometry>
-				<mesh filename="package://msd_bot/meshes/hullassm.stl" />
+				<mesh filename="file://$(find msd_bot)/meshes/hullassm.stl" />
 			</geometry>
 			<material name="hullassm_material">
@@ -20,5 +20,5 @@
 			<origin xyz="0 0 0" rpy="0 -0 0" />
 			<geometry>
-				<mesh filename="package://msd_bot/meshes/hullassm.stl" />
+				<mesh filename="file://$(find msd_bot)/meshes/hullassm.stl" />
 			</geometry>
 		</collision>
@@ -37,5 +37,5 @@
 			<origin xyz="0 0 0" rpy="0 -0 0" />
 			<geometry>
-				<mesh filename="package://msd_bot/meshes/propeller.stl" />
+				<mesh filename="file://$(find msd_bot)/meshes/propeller.stl" />
 			</geometry>
 			<material name="propeller_material">
@@ -46,5 +46,5 @@
 			<origin xyz="0 0 0" rpy="0 -0 0" />
 			<geometry>
-				<mesh filename="package://msd_bot/meshes/propeller.stl" />
+				<mesh filename="file://$(find msd_bot)/meshes/propeller.stl" />
 			</geometry>
 		</collision>
@@ -71,5 +71,5 @@
 			<origin xyz="0 0 0" rpy="0 -0 0" />
 			<geometry>
-				<mesh filename="package://msd_bot/meshes/topassm.stl" />
+				<mesh filename="file://$(find msd_bot)/meshes/topassm.stl" />
 			</geometry>
 			<material name="topassm_material">
@@ -80,5 +80,5 @@
 			<origin xyz="0 0 0" rpy="0 -0 0" />
 			<geometry>
-				<mesh filename="package://msd_bot/meshes/topassm.stl" />
+				<mesh filename="file://$(find msd_bot)/meshes/topassm.stl" />
 			</geometry>
 		</collision>
@@ -105,5 +105,5 @@
 			<origin xyz="0 0 0" rpy="0 -0 0" />
 			<geometry>
-				<mesh filename="package://msd_bot/meshes/servocargoassm.stl" />
+				<mesh filename="file://msd_bot/meshes/servocargoassm.stl" />
 			</geometry>
 			<material name="servocargoassm_material">
@@ -114,5 +114,5 @@
 			<origin xyz="0 0 0" rpy="0 -0 0" />
 			<geometry>
-				<mesh filename="package://msd_bot/meshes/servocargoassm.stl" />
+				<mesh filename="file://msd_bot/meshes/servocargoassm.stl" />
 			</geometry>
 		</collision>
@@ -125,5 +125,5 @@
 	</link>
 	<gazebo reference="servocargoassm">
-        <material>Gazebo/LightBlue  </material>
+        <material>Gazebo/Blue  </material>
     </gazebo>
 	<link name="rudder">
@@ -131,5 +131,5 @@
 			<origin xyz="0 0 0" rpy="0 -0 0" />
 			<geometry>
-				<mesh filename="package://msd_bot/meshes/rudder.stl" />
+				<mesh filename="file://$(find msd_bot)/meshes/rudder.stl" />
 			</geometry>
 			<material name="rudder_material">
@@ -140,5 +140,5 @@
 			<origin xyz="0 0 0" rpy="0 -0 0" />
 			<geometry>
-				<mesh filename="package://msd_bot/meshes/rudder.stl" />
+				<mesh filename="file://$(find msd_bot)/meshes/rudder.stl" />
 			</geometry>
 		</collision>

Commit message: centered rudder initial state

File: description/robot.urdf.xacro (robot description, xacro)
@@ -154,5 +154,5 @@
     </gazebo>
 	<joint name="servo_rudder" type="continuous">
-		<origin xyz="3.43338e-16 -0.005715 0.074295" rpy="1.5708 1.43827 -1.03735e-13" />
+		<origin xyz="3.43338e-16 -0.005715 0.074295" rpy="1.5708 0 -1.03735e-13" />
 		<parent link="servocargoassm" />
 		<child link="rudder" />

Commit message: fixed initally broken cargoassm mesh link

File: description/robot.urdf.xacro (robot description, xacro)
@@ -1,4 +1,6 @@
 <?xml version="1.0"?>
 <robot xmlns:xacro="http://www.ros.org/wiki/xacro" name="msd_bot">
+<!-- NOTE that ROS2 VSCode requires package://msd_bot for URDF \
+	preview instad of file://$(find msd_bot) but that breaks Gazebo -->
 	<link name="base_link"></link>
 	<joint name="base_link_to_base" type="fixed">
@@ -105,5 +107,5 @@
 			<origin xyz="0 0 0" rpy="0 -0 0" />
 			<geometry>
-				<mesh filename="file://msd_bot/meshes/servocargoassm.stl" />
+				<mesh filename="file://$(find msd_bot)/meshes/servocargoassm.stl" />
 			</geometry>
 			<material name="servocargoassm_material">
@@ -114,5 +116,5 @@
 			<origin xyz="0 0 0" rpy="0 -0 0" />
 			<geometry>
-				<mesh filename="file://msd_bot/meshes/servocargoassm.stl" />
+				<mesh filename="file://$(find msd_bot)/meshes/servocargoassm.stl" />
 			</geometry>
 		</collision>
