Commit message: updated o2r

File: onshape-to-robot/simplecraftv1/robot.urdf (robot description, URDF)
Before this commit: robot onshape, 4 links, 3 joints
Links:
- removed link staticrobot
- added link hullassm, mass 6.29782; collision mesh filename=package://msd_bot/hullassm_collision.stl; visual mesh filename=package://msd_bot/hullassm_visual.stl
- added link servocargoassm, mass 8.22292; collision mesh filename=package://msd_bot/servocargoassm_collision.stl; visual mesh filename=package://msd_bot/servocargoassm_visual.stl
- added link topassm, mass 0.69925; collision mesh filename=package://msd_bot/topassm_collision.stl; visual mesh filename=package://msd_bot/topassm_visual.stl
- link propeller: geometry collision mesh filename=package://msd_bot/propeller_collision.stl; visual mesh filename=package://msd_bot/propeller_visual.stl
- link rudder: geometry collision mesh filename=package://msd_bot/rudder_collision.stl; visual mesh filename=package://msd_bot/rudder_visual.stl
Joints:
- added joint hull_cargo: type fixed, parent hullassm, child servocargoassm, origin xyz=-2.77556e-17 0.3556 0.3048 rpy=-1.5708 -0 -4.62274e-32, axis 0 0 1, limit effort=1 velocity=20
- added joint hull_cover: type fixed, parent hullassm, child topassm, origin xyz=-0.2286 0.360045 0.3048 rpy=0 3.08149e-32 -4.62274e-32, axis 0 0 1, limit effort=1 velocity=20
- joint base_link_to_base: child staticrobot -> hullassm
- joint propeller_shaft: origin xyz=0.0819412 1.169 0.338466 rpy=1.5708 -1.02461e-33 -3.55271e-15 -> xyz=-2.11292e-18 0.385445 0.0889 rpy=1.5708 -0.187437 -3.49069e-15; parent staticrobot -> hullassm
- joint servo_rudder: origin xyz=0.0819412 1.21345 0.560081 rpy=7.78435e-16 6.85351e-15 0.0697974 -> xyz=3.43338e-16 -0.005715 0.074295 rpy=1.5708 1.43827 -1.03735e-13; parent staticrobot -> servocargoassm

Commit message: defined URDF using onshape models (#1)
* added basic output of onshape to urdf conversion

* added meshes

* added xacro macros of stl files

* formatted XML

* partially complete better xacro

* moved stl files to meshes folder

* added meshes to share

* simplified significantly to get minimal simulatable example

* attempted fixE ISSue with minimal example

* additional incremental test fixes

* made hull appear for vscode ROS

* just want to see the new meshes

* eliminated duplicate meshes

* consolidated subassems, made working urdf

* updated o2r

* replaced meshes with ones in the correct orientation

* removed unused meshes

* updated gazebo color tags

* changed links to meshes for Gazebo to work

* centered rudder initial state

* fixed initally broken cargoassm mesh link

---------

Co-authored-by: Atticus Russell <atticurussell@gmail.com>

File: onshape-to-robot/simplecraftv1/robot.urdf (robot description, URDF)
Before this commit: robot msd_bot, 6 links, 5 joints
Links:
- link hullassm: geometry collision mesh filename=package://msd_bot/hullassm_collision.stl; visual mesh filename=package://msd_bot/hullassm_visual.stl
- link propeller: geometry collision mesh filename=package://msd_bot/propeller_collision.stl; visual mesh filename=package://msd_bot/propeller_visual.stl
- link rudder: geometry collision mesh filename=package://msd_bot/rudder_collision.stl; visual mesh filename=package://msd_bot/rudder_visual.stl
- link servocargoassm: geometry collision mesh filename=package://msd_bot/servocargoassm_collision.stl; visual mesh filename=package://msd_bot/servocargoassm_visual.stl
- link topassm: geometry collision mesh filename=package://msd_bot/topassm_collision.stl; visual mesh filename=package://msd_bot/topassm_visual.stl
Joints:
- joint propeller_shaft: type continuous -> revolute
- joint servo_rudder: origin xyz=3.43338e-16 -0.005715 0.074295 rpy=1.5708 0 -1.03735e-13 -> xyz=3.43338e-16 -0.005715 0.074295 rpy=1.5708 1.43827 -1.03735e-13; type continuous -> revolute
